File: plane_top_view/plane.kicad_pcb (KiCad board)
At the start: 2 copper layers, 155.1 x 129.4 mm, 20 parts

Commit message: made it less jank
Parts:
- removed ? (x10): , 
- removed REF** (x2): TestPoint_Loop_D1.80mm_Drill1.0mm_Beaded, TestPoint:TestPoint_Loop_D1.80mm_Drill1.0mm_Beaded
- added TP2: TestPoint, Connector_Wire:SolderWire-0.1sqmm_1x01_D0.4mm_OD1mm, F.Cu at (99.1, 115.6)
- added TP3: TestPoint, Connector_Wire:SolderWire-0.1sqmm_1x01_D0.4mm_OD1mm, F.Cu at (99.1, 129.5)
- D3, D4: value IR26-21C_L110_TR8 -> LED; footprint LED_SMD:LED_0201_0603Metric -> LED_SMD:LED_0805_2012Metric
- moved D3 0.45 mm to (32.0, 99.5)
Routing:
- net +3V0: track 242.4 -> 310.3 mm
- net Net-(D3-K): track 111.8 -> 112.4 mm
- net GND: vias 0 -> 16
Other:
- board size 155.1 x 129.4 mm -> 155 x 129.4 mm
