File: plane_top_view/plane.kicad_sch (KiCad schematic)
At the start: 8 parts

Commit message: made it less jank
Parts:
- removed D3, D4: IR26-21C_L110_TR8, LED_SMD:LED_0201_0603Metric, symbol LED:IR26-21C_L110_TR8
- added D3, D4: LED, LED_SMD:LED_0805_2012Metric, symbol Device:LED
- added TP2, TP3: TestPoint, MountingHole:MountingHole_2.2mm_M2_Pad_TopBottom, symbol Connector:TestPoint
Connections:
- net +3V0: now also D3.2 (A), D4.2 (A), TP2.1
- net GND: now also TP3.1
- net at R4.1: now also D4.1 (K)
- net at R3.1: now also D3.1 (K)
